Commit message: Version 2

File: src/waypoint_follower/config/robot.urdf (robot description, URDF)
Before this commit: robot autonomous_waypoint_follower, 6 links, 5 joints
Links:
- added link camera_link, mass 0.05; visual box size=0.04 0.08 0.04
- link base_link: mass ${chassis_mass} -> 12.0; geometry collision box size=0.8 0.5 0.4; visual box size=0.7 0.4 0.05
- link caster_wheel: mass ${caster_mass} -> 0.3; geometry collision sphere radius=0.07; visual sphere radius=0.07
- link laser_link: mass 0.05 -> 0.08; geometry collision cylinder length=0.07 radius=0.03; visual cylinder length=0.07 radius=0.03
- link left_wheel: mass ${wheel_mass} -> 1.0; geometry collision cylinder length=0.12 radius=0.15; visual cylinder length=0.096 radius=0.16
- link right_wheel: mass ${wheel_mass} -> 1.0; geometry collision cylinder length=0.12 radius=0.15; visual cylinder length=0.096 radius=0.16
Joints:
- added joint camera_joint: type fixed, parent base_link, child camera_link, origin xyz=0.325 0 0.2 rpy=0 0 0
- joint caster_wheel_joint: origin xyz=${chassis_length/2 - caster_radius} 0 ${-chassis_height/2 + caster_radius} rpy=0 0 0 -> xyz=0.33 0 -0.13 rpy=0 0 0
- joint imu_joint: origin xyz=0 0 0 rpy=0 0 0 -> xyz=0 0 0.2 rpy=0 0 0
- joint laser_joint: origin xyz=${chassis_length/2 - 0.05} 0 ${chassis_height/2 + 0.05} rpy=0 0 0 -> xyz=0.3 0 0.25 rpy=0 0 0
- joint left_wheel_joint: origin xyz=0 ${wheel_separation/2} ${-chassis_height/2 + wheel_radius} rpy=0 0 0 -> xyz=0 0.2 -0.05 rpy=0 0 0
- joint right_wheel_joint: origin xyz=0 ${-wheel_separation/2} ${-chassis_height/2 + wheel_radius} rpy=0 0 0 -> xyz=0 -0.2 -0.05 rpy=0 0 0

Commit message: Version 1

File: src/waypoint_follower/config/robot.urdf (robot description, URDF)
Before this commit: robot autonomous_waypoint_follower, 7 links, 6 joints
Joints:
- joint camera_joint: origin xyz=0.325 0 0.2 rpy=0 0 0 -> xyz=0.4 0 0.1 rpy=0 0.2 0
- joint caster_wheel_joint: origin xyz=0.33 0 -0.13 rpy=0 0 0 -> xyz=0.35 0 -0.17 rpy=0 0 0
- joint imu_joint: origin xyz=0 0 0.2 rpy=0 0 0 -> xyz=0 0 0 rpy=0 0 0
- joint laser_joint: origin xyz=0.3 0 0.25 rpy=0 0 0 -> xyz=0 0 0.25 rpy=0 0 0
